File: Eagle/LDBiasDriver.brd (EAGLE design)
At the start: 44.8 x 22.9 mm, 23 parts, among them IC1 MCP1703-5002E/DB, IC2 MLD203P1, IC3 LM358D

Commit message: used a standard connector spacing for the SMA alternative.
Parts:
- added LD2: (no value), pinhead:1X02
Connections:
- net N$10: now also LD2.1
- net N$8: now also LD2.2
Routing:
- net N$10: track 10.3 -> 12.2 mm
- net N$8: track 4.37 -> 5.66 mm
Changed lines of the file:
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@@
 <element name="LED1" library="led" package="CHIPLED_1206" value="" x="10.795" y="6.35" rot="R90"/>
 <element name="R2" library="rcl" package="R0805" value="1k" x="14.605" y="10.795" rot="R90"/>
+<element name="LD2" library="pinhead" package="1X02" value="" x="41.91" y="9.2075" rot="R270"/>
 </elements>
 <signals>
@@
 <contactref element="R3" pad="2"/>
 <contactref element="LD" pad="1"/>
-<wire x1="37.78" y1="6.35" x2="41.2496" y2="6.35" width="1.016" layer="1"/>
+<wire x1="37.78" y1="6.35" x2="40.64" y2="6.35" width="1.016" layer="1"/>
+<wire x1="40.64" y1="6.35" x2="41.2496" y2="6.35" width="1.016" layer="1"/>
 <wire x1="41.2496" y1="6.35" x2="41.8846" y2="6.985" width="1.016" layer="1"/>
+<contactref element="LD2" pad="2"/>
+<wire x1="40.64" y1="6.0325" x2="40.64" y2="6.35" width="0.4064" layer="1"/>
+<wire x1="41.91" y1="7.9375" x2="41.8846" y2="7.9375" width="0.4064" layer="1"/>
+<wire x1="41.8846" y1="7.9375" x2="41.8846" y2="6.985" width="0.4064" layer="1"/>
 </signal>
 <signal name="N$10">
@@
 <wire x1="41.91" y1="14.2875" x2="41.91" y2="11.43" width="0.3556" layer="1"/>
 <wire x1="41.91" y1="11.43" x2="41.8846" y2="11.4046" width="0.3556" layer="1"/>
+<contactref element="LD2" pad="1"/>
+<wire x1="41.8846" y1="3.4925" x2="41.8846" y2="2.5654" width="0.4064" layer="1"/>
+<wire x1="41.91" y1="10.4775" x2="41.8846" y2="10.4775" width="0.4064" layer="1"/>
+<wire x1="41.8846" y1="10.4775" x2="41.8846" y2="11.4046" width="0.4064" layer="1"/>
+<wire x1="41.8846" y1="11.43" x2="41.8846" y2="11.4046" width="0.4064" layer="1"/>
 <wire x1="41.8846" y1="11.4046" x2="41.8846" y2="11.4046" width="0" layer="19" extent="1-16"/>
-<wire x1="41.8846" y1="2.5654" x2="41.8846" y2="11.4046" width="0" layer="19" extent="1-16"/>
+<wire x1="41.8846" y1="3.4925" x2="41.91" y2="10.4775" width="0" layer="19" extent="1-1"/>
 <wire x1="41.8846" y1="2.5654" x2="41.8846" y2="2.5654" width="0" layer="19" extent="1-16"/>
 </signal>
@@
 <wire x1="13.97" y1="19.685" x2="8.255" y2="19.685" width="0.8128" layer="1"/>
 </signal>
-<signal name="N$20">
-<via x="40.3225" y="7.14375" extent="1-16" drill="1" diameter="1.778"/>
-</signal>
-<signal name="N$21">
-<via x="40.3225" y="2.69875" extent="1-16" drill="1" diameter="1.778"/>
-</signal>
 </signals>

Commit message: Updates based on experience
Parts:
- LD: value SMA-142-0701-871/876 -> SMA-142-0711-821/826; device con-coax:J502-ND-142-0701-871/876 -> con-coax:J502-ND-142-0711-821/826
- moved LD2 1.75 mm to (40.8, 7.86)
- moved LD 0.64 mm to (44.5, 6.35)
- moved PD 0.40 mm to (41.9, 15.2)
Routing:
- net N$10: track 12.2 -> 18.8 mm
- net N$8: track 5.66 -> 6.43 mm
- net N$2: track 28.1 -> 27.4 mm
Changed lines of the file:
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@@
 <setting verticaltext="up"/>
 </settings>
-<grid distance="0.05" unitdist="inch" unit="mm" style="lines" multiple="1" display="no" altdistance="0.00625" altunitdist="inch" altunit="inch"/>
+<grid distance="0.05" unitdist="inch" unit="mm" style="lines" multiple="1" display="no" altdistance="3.125" altunitdist="mil" altunit="mil"/>
 <layers>
 <layer number="1" name="Top" color="4" fill="1" visible="yes" active="yes"/>
@@
 <attribute name="MPN" value="237-102" x="2.54" y="17.145" size="1.778" layer="27" rot="R90" display="off"/>
 </element>
-<element name="LD" library="con-coax" package="J502-ND-142-0701-871/876" value="SMA-142-0701-871/876" x="44.45" y="6.985" rot="R180">
-<attribute name="MF" value="JOHNSON COMPONENTS" x="44.45" y="6.985" size="1.778" layer="27" rot="R180" display="off"/>
-<attribute name="OC_NEWARK" value="91B6105" x="44.45" y="6.985" size="1.778" layer="27" rot="R180" display="off"/>
-<attribute name="OC_FARNELL" value="1339835" x="44.45" y="6.985" size="1.778" layer="27" rot="R180" display="off"/>
-<attribute name="MPN" value="142-0701-871" x="44.45" y="6.985" size="1.778" layer="27" rot="R180" display="off"/>
+<element name="LD" library="con-coax" package="J502-ND-142-0711-821/826" value="SMA-142-0711-821/826" x="44.45" y="6.35" rot="R180">
+<attribute name="MF" value="JOHNSON COMPONENTS" x="44.45" y="6.35" size="1.778" layer="27" rot="R180" display="off"/>
+<attribute name="OC_NEWARK" value="16F3627" x="44.45" y="6.35" size="1.778" layer="27" rot="R180" display="off"/>
+<attribute name="OC_FARNELL" value="1019328" x="44.45" y="6.35" size="1.778" layer="27" rot="R180" display="off"/>
+<attribute name="MPN" value="142-0711-821" x="44.45" y="6.35" size="1.778" layer="27" rot="R180" display="off"/>
 </element>
 <element name="IC2" library="laser diode" package="MLD203" value="MLD203P1" x="17.78" y="15.875"/>
-<element name="PD" library="pinhead" package="1X02" value="" x="41.91" y="15.5575" rot="R270"/>
+<element name="PD" library="pinhead" package="1X02" value="" x="41.91" y="15.160625" rot="R270"/>
 <element name="R4" library="pot" package="RJ9W" value="100k" x="36.195" y="20.32" rot="R180"/>
 <element name="C3" library="rcl" package="C0805" value="100pF" x="38.1" y="14.605" rot="R270"/>
@@
 <element name="LED1" library="led" package="CHIPLED_1206" value="" x="10.795" y="6.35" rot="R90"/>
 <element name="R2" library="rcl" package="R0805" value="1k" x="14.605" y="10.795" rot="R90"/>
-<element name="LD2" library="pinhead" package="1X02" value="" x="41.91" y="9.2075" rot="R270"/>
+<element name="LD2" library="pinhead" package="1X02" value="" x="40.79875" y="7.858125" rot="R270"/>
 </elements>
 <signals>
@@
 <vertex x="0" y="0"/>
 </polygon>
-<polygon width="0.6096" layer="16">
+<polygon width="0.4064" layer="16">
 <vertex x="-1.27" y="22.86"/>
 <vertex x="0" y="0"/>
@@
 <via x="12.7" y="16.8275" extent="1-16" drill="0.5"/>
 <contactref element="IC2" pad="P$3"/>
-<via x="19.685" y="13.6525" extent="1-16" drill="0.5"/>
+<via x="16.271875" y="13.335" extent="1-16" drill="0.5"/>
 </signal>
 <signal name="N$2">
@@
 <wire x1="22.225" y1="9.525" x2="30.1625" y2="17.4625" width="0.3556" layer="16"/>
 <wire x1="30.1625" y1="17.4625" x2="30.1625" y2="20.6375" width="0.3556" layer="16"/>
-<wire x1="30.1625" y1="20.6375" x2="29.36875" y2="21.43125" width="0.3556" layer="16"/>
-<wire x1="29.36875" y1="21.43125" x2="26.19375" y2="21.43125" width="0.3556" layer="16"/>
-<wire x1="26.19375" y1="21.43125" x2="26.035" y2="21.2725" width="0.3556" layer="16"/>
-<wire x1="26.035" y1="21.2725" x2="26.035" y2="19.685" width="0.3556" layer="16"/>
+<wire x1="30.1625" y1="20.6375" x2="29.448125" y2="21.351875" width="0.3556" layer="16"/>
+<wire x1="29.448125" y1="21.351875" x2="27.225625" y2="21.351875" width="0.3556" layer="16"/>
+<wire x1="27.225625" y1="21.351875" x2="26.035" y2="20.16125" width="0.3556" layer="16"/>
+<wire x1="26.035" y1="20.16125" x2="26.035" y2="19.685" width="0.3556" layer="16"/>
 </signal>
 <signal name="N$4">
@@
 <contactref element="LD" pad="1"/>
 <wire x1="37.78" y1="6.35" x2="40.64" y2="6.35" width="1.016" layer="1"/>
-<wire x1="40.64" y1="6.35" x2="41.2496" y2="6.35" width="1.016" layer="1"/>
-<wire x1="41.2496" y1="6.35" x2="41.8846" y2="6.985" width="1.016" layer="1"/>
+<wire x1="40.64" y1="6.35" x2="42.3346" y2="6.35" width="1.016" layer="1"/>
 <contactref element="LD2" pad="2"/>
 <wire x1="40.64" y1="6.0325" x2="40.64" y2="6.35" width="0.4064" layer="1"/>
-<wire x1="41.91" y1="7.9375" x2="41.8846" y2="7.9375" width="0.4064" layer="1"/>
-<wire x1="41.8846" y1="7.9375" x2="41.8846" y2="6.985" width="0.4064" layer="1"/>
+<wire x1="40.79875" y1="6.588125" x2="41.72585" y2="6.50875" width="0.4064" layer="1"/>
+<wire x1="41.72585" y1="6.50875" x2="42.3346" y2="6.35" width="0.4064" layer="1"/>
 </signal>
 <signal name="N$10">
@@
 <contactref element="PD" pad="2"/>
 <wire x1="34.78" y1="12.065" x2="36.195" y2="12.065" width="1.016" layer="1"/>
-<wire x1="36.195" y1="12.065" x2="36.83" y2="11.43" width="1.016" layer="1"/>
-<wire x1="36.83" y1="11.43" x2="41.8592" y2="11.43" width="1.016" layer="1"/>
-<wire x1="41.8592" y1="11.43" x2="41.8846" y2="11.4046" width="1.016" layer="1"/>
-<wire x1="41.91" y1="14.2875" x2="41.91" y2="11.43" width="0.3556" layer="1"/>
-<wire x1="41.91" y1="11.43" x2="41.8846" y2="11.4046" width="0.3556" layer="1"/>
+<wire x1="36.195" y1="12.065" x2="38.1" y2="10.16" width="1.016" layer="1"/>
+<wire x1="38.1" y1="10.16" x2="43.1292" y2="10.16" width="1.016" layer="1"/>
+<wire x1="43.1292" y1="10.16" x2="42.3346" y2="9.8446" width="1.016" layer="1"/>
+<wire x1="41.91" y1="13.890625" x2="41.91" y2="9.763125" width="0.3556" layer="1"/>
+<wire x1="41.91" y1="9.763125" x2="42.3346" y2="9.8446" width="0.3556" layer="1"/>
 <contactref element="LD2" pad="1"/>
-<wire x1="41.8846" y1="3.4925" x2="41.8846" y2="2.5654" width="0.4064" layer="1"/>
-<wire x1="41.91" y1="10.4775" x2="41.8846" y2="10.4775" width="0.4064" layer="1"/>
-<wire x1="41.8846" y1="10.4775" x2="41.8846" y2="11.4046" width="0.4064" layer="1"/>
-<wire x1="41.8846" y1="11.43" x2="41.8846" y2="11.4046" width="0.4064" layer="1"/>
-<wire x1="41.8846" y1="11.4046" x2="41.8846" y2="11.4046" width="0" layer="19" extent="1-16"/>
-<wire x1="41.8846" y1="3.4925" x2="41.91" y2="10.4775" width="0" layer="19" extent="1-1"/>
-<wire x1="41.8846" y1="2.5654" x2="41.8846" y2="2.5654" width="0" layer="19" extent="1-16"/>
+<wire x1="41.8846" y1="3.4925" x2="42.3346" y2="2.8554" width="0.4064" layer="1"/>
+<wire x1="40.79875" y1="9.128125" x2="41.8846" y2="10.4775" width="0.4064" layer="1"/>
+<wire x1="41.8846" y1="10.4775" x2="42.3346" y2="9.8446" width="0.4064" layer="1"/>
+<wire x1="42.04335" y1="10.715625" x2="42.3346" y2="9.8446" width="0.4064" layer="1"/>
+<wire x1="42.3346" y1="9.8446" x2="42.3346" y2="9.8446" width="0" layer="19" extent="1-16"/>
+<wire x1="41.8846" y1="3.4925" x2="40.79875" y2="9.128125" width="0" layer="19" extent="1-1"/>
+<wire x1="42.3346" y1="2.8554" x2="42.3346" y2="2.8554" width="0" layer="19" extent="1-16"/>
 </signal>
 <signal name="N$11">
@@
 <wire x1="37.1475" y1="16.8275" x2="41.275" y2="16.8275" width="0.3556" layer="1"/>
 <wire x1="41.275" y1="16.8275" x2="41.5925" y2="17.145" width="0.3556" layer="1"/>
-<wire x1="41.5925" y1="17.145" x2="41.91" y2="16.8275" width="0.3556" layer="1"/>
+<wire x1="41.5925" y1="17.145" x2="41.91" y2="16.430625" width="0.3556" layer="1"/>
 </signal>
 <signal name="N$12">
@@
 <wire x1="15.0114" y1="18.1864" x2="15.875" y2="19.05" width="0.8128" layer="1"/>
 <wire x1="15.875" y1="19.05" x2="15.875" y2="20.955" width="0.8128" layer="1"/>
-<wire x1="17.78" y1="15.875" x2="17.78" y2="14.605" width="0.8128" layer="1"/>
 <wire x1="15.0114" y1="14.6812" x2="15.0114" y2="12.1514" width="0.3556" layer="1"/>
 <wire x1="15.0114" y1="12.1514" x2="14.605" y2="11.745" width="0.6096" layer="1"/>
@@
 <wire x1="17.30625" y1="21.2725" x2="17.465" y2="21.43125" width="0.8128" layer="1"/>
 <wire x1="17.465" y1="21.43125" x2="17.465" y2="19.05" width="0.8128" layer="1"/>
+<wire x1="17.78" y1="15.875" x2="17.78" y2="14.605" width="0.6096" layer="1"/>
 </signal>
 <signal name="N$16">
