File: Controller/BiasController/BiasController.brd (EAGLE design)
At the start: 88.7 x 47 mm, 32 parts, among them IC1 4066D, X4 IN-A, X5 IN-B

Commit message: controller done but going to change
Parts:
- removed U$3: NANO, Arduino-clone:NANO
- added C8: 10u, rcl:C0805
- added IC2: REG1117, burr-brown:SOT223
- added IC4: (no value), v-reg:78XXS
- moved X4 2.54 mm to (27.9, 0.00)
- moved X1 1.42 mm to (4.45, 7.62)
Connections:
- new net V+: C8.1, IC2.2, IC4.OUT, X1.2
- net +12V: now also IC2.3, IC4.IN
- net GND: now also C8.2, IC2.1, IC4.GND, X1.1; no longer X1.2
- net N$9: no longer X1.1
Routing:
- net V+: track 0.00 -> 18.6 mm, vias 0 -> 1
- net N$9: track 30.4 -> 13.1 mm
- net +12V: track 94.4 -> 106.3 mm, vias 1 -> 0
- net N$13: track 4.55 -> 6.16 mm
Other:
- board text added: "+5-16V In"
- board text added: "5V Out"
- board text removed: "5-16V"
- board text removed: "GND"

Commit message: final version as manufactured
Parts:
- removed C4: 0.1u, rcl:C0805
- removed U$6: MCP4251-103E/SL, Custom:SOIC127P600X175-14N
- added C10, C9: 0.1u, rcl:C0805
- added R10: 4.7k, rcl:R0805
- added U1: MCP4726A0, SparkFun-AnalogIC:SOT23-6
- added U2: MCP4726A1, SparkFun-AnalogIC:SOT23-6
- added X2: (no value), con-wago-500:W237-102
- R2: value 10k -> 4.7k
- moved R1 26.7 mm to (72.4, 34.9), turned to 90 degrees
- moved R2 24.3 mm to (57.1, 11.4), turned to 90 degrees
- moved U$1 24.1 mm to (45.7, 24.1)
- moved U$2 24.1 mm to (45.7, 0.00)
- moved C3 19.3 mm to (67.9, 29.8), turned to 270 degrees
- moved U$5 17.3 mm to (73.7, 26.7)
- moved R6 12.7 mm to (41.9, 33.0)
- moved C5 3.31 mm to (54.6, 28.6)
- moved IC1 3.24 mm to (61.0, 26.7)
Connections:
- removed net CSB: JP2.13, U$6.1
- removed net N$5: U$5.6, U$5.8
- removed net N$6 (its old number): IC1.10, IC1.9, U$6.7
- removed net N$8: U$2.C, U$6.9
- removed net SHDNB: JP2.11, R2.1, U$6.12
- new net N$19: IC1.1, U2.1
- new net N$20: U$2.B, U$5.6
- new net N$4: IC1.10, IC1.9, U$5.8
- new net SCL: JP1.7, R2.2, U1.5, U2.5
- new net SDA: JP1.8, R10.2, U1.4, U2.4
- net +5V: now also C10.2, C9.2, R10.1, R2.1, U1.3, U2.3; no longer C4.2, U$6.14
- net BUTTON: now also JP1.9; no longer JP1.8
- net CSA: now also JP2.13; no longer JP2.12
- net EX-A: now also IC1.12, JP2.10; no longer IC1.5, JP2.5
- net EX-B: now also IC1.5; no longer IC1.12
- net GND: now also C10.1, C9.1, U$5.5, U1.2, U2.2, X2.2; no longer C4.1, R2.2, U$6.10, U$6.4
- net IN-A: now also IC1.11, JP2.11; no longer IC1.4, JP1.7
- net IN-B: now also IC1.4; no longer IC1.11
- net LED: now also JP1.10; no longer JP1.9
- net N$1: now also U$1.C, U1.6; no longer IC1.1, U$1.B
- net N$2: now also U1.1; no longer U$2.B
- net N$3: now also U$1.B; no longer U$1.C
- net N$7: now also U$2.C, U2.6; no longer U$6.6, U$6.8
- net N$9: now also X2.1
- net NEX-A: now also IC1.6; no longer IC1.13
- net NEX-B: now also IC1.13; no longer IC1.6
- net SCK: no longer U$6.2
- net SDI: no longer U$6.3
- net SDO: no longer U$6.13
- net SHDNA: no longer JP2.10
Routing:
- net SDA: track 0.00 -> 102.2 mm, vias 0 -> 2
- net SCL: track 0.00 -> 93.4 mm, vias 0 -> 2
- net SHDNA: track 66.4 -> 4.94 mm
- net SHDNB: track 37.3 -> 0.00 mm, vias 2 -> 0
- net CSB: track 36.2 -> 0.00 mm
- net VMONB: track 36.9 -> 61.1 mm, vias 0 -> 2
- net VMONA: track 60.9 -> 37.1 mm, vias 2 -> 1
- net N$6 (its old number): track 21.1 -> 0.00 mm, vias 2 -> 0
- net N$4: track 0.00 -> 20.3 mm
- net +5V: track 95.1 -> 112.7 mm, vias 6 -> 7
- net N$2: track 20.4 -> 3.88 mm, vias 1 -> 0
- net N$7: track 5.25 -> 19.0 mm
- net NEX-A: track 25.9 -> 39.0 mm
- net SDO: track 59.2 -> 47.0 mm, vias 0 -> 1
- net SDI: track 67.9 -> 56.8 mm, vias 0 -> 1
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Other:
- outline, holes or cut-outs redrawn
- board text added: "Vbias = 2.5 x DAC x DIV"
- board text added: "Vbias = Vin x DIV"
- board text removed: "BTN"
- board text removed: "CSA"
- board text removed: "CSB"
- board text removed: "EX-A"
- board text removed: "EX-B"
- board text removed: "IN-A"
- board text removed: "IN-B"
- board text removed: "LED"
- board text removed: "MONA"
- board text removed: "MONB"
- board text removed: "NEX-A"
- board text removed: "NEX-B"
- board text removed: "SHDNA"
- board text removed: "SHDNB"
