File: Controller/BiasController/BiasController.sch (EAGLE design)
At the start: 32 parts, among them IC1 4066D, X4 IN-A, X5 IN-B

Commit message: controller done but going to change
Parts:
- removed U$3: NANO, Arduino-clone:NANO
- added C8: 10u, rcl:C-EUC0805
- added IC2: REG1117, burr-brown:REG1117
- added IC4: (no value), v-reg:78XXS
Connections:
- new net V+: C8.1, IC2.VOUT, IC4.OUT, X1-2.KL
- net +12V: now also IC2.VIN, IC4.IN
- net GND: now also C8.2, IC2.GND, IC4.GND, X1-1.KL; no longer X1-2.KL
- net N$9: no longer X1-1.KL
Other:
- moved on the sheet: X1-1, X1-2
Changed lines of the file:
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@@
 <part name="U$5" library="Custom" deviceset="MCP4251-103E/SL" device=""/>
 <part name="U$6" library="Custom" deviceset="MCP4251-103E/SL" device=""/>
-<part name="X1" library="con-wago-500" deviceset="W237-102" device=""/>
 <part name="J1" library="con-jack" deviceset="JACK-PLUG" device="0"/>
 <part name="C2" library="rcl" deviceset="C-EU" device="C0805" value="0.1u"/>
@@
 <part name="JP1" library="SparkFun-Connectors" deviceset="M15" device="LOCK_LONGPADS"/>
 <part name="JP2" library="SparkFun-Connectors" deviceset="M15" device="LOCK_LONGPADS"/>
-<part name="U$3" library="Arduino-clone" deviceset="NANO" device=""/>
 <part name="S1" library="SparkFun" deviceset="TAC_SWITCH" device="PTH"/>
 <part name="LED1" library="SparkFun" deviceset="LED" device="0603"/>
@@
 <part name="GND16" library="supply1" deviceset="GND" device=""/>
 <part name="C1" library="rcl" deviceset="C-EU" device="C0805" value="10u"/>
+<part name="IC2" library="burr-brown" deviceset="REG1117" device=""/>
+<part name="IC4" library="v-reg" deviceset="78XXS" device=""/>
+<part name="P+11" library="supply1" deviceset="+12V" device=""/>
+<part name="GND17" library="supply1" deviceset="GND" device=""/>
+<part name="GND18" library="supply1" deviceset="GND" device=""/>
+<part name="P+12" library="supply1" deviceset="V+" device=""/>
+<part name="C8" library="rcl" deviceset="C-EU" device="C0805" value="10u"/>
+<part name="X1" library="con-wago-500" deviceset="W237-102" device=""/>
+<part name="GND19" library="supply1" deviceset="GND" device=""/>
+<part name="GND20" library="supply1" deviceset="GND" device=""/>
 </parts>
 <sheets>
@@
 <instance part="U$5" gate="A" x="83.82" y="76.2"/>
 <instance part="U$6" gate="A" x="83.82" y="12.7"/>
-<instance part="X1" gate="-1" x="68.58" y="193.04"/>
-<instance part="X1" gate="-2" x="68.58" y="187.96"/>
 <instance part="J1" gate="G$1" x="68.58" y="175.26"/>
 <instance part="C2" gate="G$1" x="106.68" y="185.42"/>
@@
 <instance part="JP1" gate="G$1" x="233.68" y="147.32" rot="MR0"/>
 <instance part="JP2" gate="G$1" x="243.84" y="147.32"/>
-<instance part="U$3" gate="G$1" x="246.38" y="203.2"/>
 <instance part="S1" gate="S" x="142.24" y="187.96"/>
 <instance part="LED1" gate="G$1" x="139.7" y="175.26" rot="R90"/>
@@
 <instance part="GND16" gate="1" x="160.02" y="170.18"/>
 <instance part="C1" gate="G$1" x="96.52" y="185.42"/>
+<instance part="IC2" gate="G$1" x="101.6" y="223.52"/>
+<instance part="IC4" gate="1" x="96.52" y="246.38"/>
+<instance part="P+11" gate="1" x="86.36" y="251.46"/>
+<instance part="GND17" gate="1" x="101.6" y="208.28"/>
+<instance part="GND18" gate="1" x="96.52" y="236.22"/>
+<instance part="P+12" gate="1" x="127" y="251.46"/>
+<instance part="C8" gate="G$1" x="116.84" y="241.3"/>
+<instance part="X1" gate="-1" x="142.24" y="241.3" rot="R180"/>
+<instance part="X1" gate="-2" x="142.24" y="246.38" rot="R180"/>
+<instance part="GND19" gate="1" x="132.08" y="233.68"/>
+<instance part="GND20" gate="1" x="116.84" y="231.14"/>
 </instances>
 <busses>
@@
 <net name="GND" class="0">
 <segment>
-<pinref part="X1" gate="-2" pin="KL"/>
-<wire x1="73.66" y1="187.96" x2="76.2" y2="187.96" width="0.1524" layer="91"/>
-<wire x1="76.2" y1="187.96" x2="76.2" y2="175.26" width="0.1524" layer="91"/>
 <pinref part="GND1" gate="1" pin="GND"/>
 <wire x1="76.2" y1="175.26" x2="76.2" y2="172.72" width="0.1524" layer="91"/>
@@
 <pinref part="J1" gate="G$1" pin="2"/>
 <wire x1="73.66" y1="175.26" x2="76.2" y2="175.26" width="0.1524" layer="91"/>
-<junction x="76.2" y="175.26"/>
 <junction x="76.2" y="172.72"/>
 <junction x="96.52" y="170.18"/>
@@
 <junction x="147.32" y="187.96"/>
 </segment>
+<segment>
+<pinref part="IC4" gate="1" pin="GND"/>
+<pinref part="GND18" gate="1" pin="GND"/>
+</segment>
+<segment>
+<pinref part="IC2" gate="G$1" pin="GND"/>
+<pinref part="GND17" gate="1" pin="GND"/>
+</segment>
+<segment>
+<pinref part="X1" gate="-1" pin="KL"/>
+<pinref part="GND19" gate="1" pin="GND"/>
+<wire x1="137.16" y1="241.3" x2="132.08" y2="241.3" width="0.1524" layer="91"/>
+<wire x1="132.08" y1="241.3" x2="132.08" y2="236.22" width="0.1524" layer="91"/>
+</segment>
+<segment>
+<pinref part="C8" gate="G$1" pin="2"/>
+<pinref part="GND20" gate="1" pin="GND"/>
+<wire x1="116.84" y1="236.22" x2="116.84" y2="233.68" width="0.1524" layer="91"/>
+</segment>
 </net>
 <net name="+12V" class="0">
@@
 <junction x="190.5" y="22.86"/>
 </segment>
+<segment>
+<pinref part="P+11" gate="1" pin="+12V"/>
+<wire x1="86.36" y1="248.92" x2="86.36" y2="246.38" width="0.1524" layer="91"/>
+<wire x1="86.36" y1="246.38" x2="86.36" y2="223.52" width="0.1524" layer="91"/>
+<pinref part="IC4" gate="1" pin="IN"/>
+<wire x1="88.9" y1="246.38" x2="86.36" y2="246.38" width="0.1524" layer="91"/>
+<pinref part="IC2" gate="G$1" pin="VIN"/>
+<wire x1="86.36" y1="223.52" x2="88.9" y2="223.52" width="0.1524" layer="91"/>
+<junction x="86.36" y="246.38"/>
+</segment>
 </net>
 <net name="+5V" class="0">
@@
 <net name="N$9" class="0">
 <segment>
-<pinref part="X1" gate="-1" pin="KL"/>
-<wire x1="73.66" y1="193.04" x2="78.74" y2="193.04" width="0.1524" layer="91"/>
 <pinref part="J1" gate="G$1" pin="3"/>
-<wire x1="73.66" y1="177.8" x2="78.74" y2="177.8" width="0.1524" layer="91"/>
-<wire x1="78.74" y1="177.8" x2="78.74" y2="193.04" width="0.1524" layer="91"/>
+<wire x1="73.66" y1="177.8" x2="76.2" y2="177.8" width="0.1524" layer="91"/>
 <pinref part="D2" gate="G$1" pin="A"/>
-<junction x="78.74" y="193.04"/>
+<wire x1="78.74" y1="193.04" x2="76.2" y2="193.04" width="0.1524" layer="91"/>
+<wire x1="76.2" y1="193.04" x2="76.2" y2="177.8" width="0.1524" layer="91"/>
 </segment>
 </net>
@@
 </segment>
 </net>
+<net name="V+" class="0">
+<segment>
+<pinref part="IC4" gate="1" pin="OUT"/>
+<pinref part="P+12" gate="1" pin="V+"/>
+<wire x1="104.14" y1="246.38" x2="116.84" y2="246.38" width="0.1524" layer="91"/>
+<wire x1="116.84" y1="246.38" x2="127" y2="246.38" width="0.1524" layer="91"/>
+<wire x1="127" y1="246.38" x2="127" y2="248.92" width="0.1524" layer="91"/>
+<wire x1="127" y1="223.52" x2="127" y2="246.38" width="0.1524" layer="91"/>
+<pinref part="IC2" gate="G$1" pin="VOUT"/>
+<junction x="127" y="246.38"/>
+<pinref part="C8" gate="G$1" pin="1"/>
+<wire x1="114.3" y1="223.52" x2="127" y2="223.52" width="0.1524" layer="91"/>
+<wire x1="116.84" y1="243.84" x2="116.84" y2="246.38" width="0.1524" layer="91"/>
+<junction x="116.84" y="246.38"/>
+<pinref part="X1" gate="-2" pin="KL"/>
+<wire x1="137.16" y1="246.38" x2="127" y2="246.38" width="0.1524" layer="91"/>
+</segment>
+</net>

Commit message: final version as manufactured
Parts:
- removed C4: 0.1u, rcl:C-EUC0805
- removed U$6: MCP4251-103E/SL, Custom:MCP4251-103E/SL
- added C10, C9: 0.1u, rcl:C-EUC0805
- added R10: 4.7k, rcl:R-EU_R0805
- added U1: MCP4726A0, SparkFun-AnalogIC:MCP4725SOT-23
- added U2: MCP4726A1, SparkFun-AnalogIC:MCP4725SOT-23
- added X2: (no value), con-wago-500:W237-102
- R2: value 10k -> 4.7k
Connections:
- removed net CSB: JP2.13, U$6.~CS
- removed net N$5: U$5.P0A, U$5.P1W
- removed net N$6 (its old number): IC1C.B, IC1D.B, U$6.P1A
- removed net N$8: U$2.C, U$6.P0W
- removed net SHDNB: JP2.11, R2.1, U$6.~SHDN
- new net N$19: IC1A.A, U2.VOUT
- new net N$20: U$2.B, U$5.P1W
- new net N$4: IC1C.B, IC1D.B, U$5.P0A
- new net SCL: JP1.7, R2.2, U1.SCL, U2.SCL
- new net SDA: JP1.8, R10.2, U1.SDA, U2.SDA
- net +5V: now also C10.2, C9.2, R10.1, R2.1, U1.VDD, U2.VDD; no longer C4.2, U$6.VDD
- net BUTTON: now also JP1.9; no longer JP1.8
- net CSA: now also JP2.13; no longer JP2.12
- net EX-A: now also IC1D.C, JP2.10; no longer IC1B.C, JP2.5
- net EX-B: now also IC1B.C; no longer IC1D.C
- net GND: now also C10.1, C9.1, U$5.P1B, U1.VSS, U2.VSS, X2-2.KL; no longer C4.1, R2.2, U$6.P0B, U$6.VSS
- net IN-A: now also IC1D.A, JP2.11; no longer IC1B.A, JP1.7
- net IN-B: now also IC1B.A; no longer IC1D.A
- net LED: now also JP1.10; no longer JP1.9
- net N$1: now also U$1.C, U1.AO; no longer IC1A.A, U$1.B
- net N$2: now also U1.VOUT; no longer U$2.B
- net N$3: now also U$1.B; no longer U$1.C
- net N$7: now also U$2.C, U2.AO; no longer U$6.P0A, U$6.P1W
- net N$9: now also X2-1.KL
- net NEX-A: now also IC1C.C; no longer IC1A.C
- net NEX-B: now also IC1A.C; no longer IC1C.C
- net SCK: no longer U$6.SCK
- net SDI: no longer U$6.SDI
- net SDO: no longer U$6.SDO
- net SHDNA: no longer JP2.10
Other:
- moved on the sheet: C3, IC1A, IC1B, IC1C, IC1D, R1, R2, R4, U$5
