File: Constant Current/Eagle/LDBiasDriver CC v2.sch (EAGLE design)
At the start: 24 parts, among them IC1 MCP1703-5002E/DB, IC3 LM358D, U1 MCP4726A0

Commit message: updates
Parts:
- removed ISENS: (no value), con-wago-500:W237-102
- added JP2: (no value), SparkFun-Connectors:M06POLAR_LOCK
- added Q1: (no value), adafruit:MOSFET-NREFLOW
- added R10, R12, R4, R9: 4.7k, rcl:R-EU_R0805
- added R11: 330, rcl:R-EU_R0805
Connections:
- removed net N$14: L1.1, VIN-1.KL
- removed net N$18: IC3A.OUT, ISENS-1.KL, R7.2
- new net ISENSE: IC3A.OUT, JP2.6, R7.2
- new net MOD: JP2.5, R11.1
- new net N$10: Q1.G, R11.2, R12.2
- new net N$13: R10.2, U1.VOUT
- new net SCL: JP2.4, R9.2, U1.SCL
- new net SDA: JP2.3, R4.2, U1.SDA
- new net VIN: JP2.2, L1.1, VIN-1.KL
- net +5V: now also R4.1, R9.1
- net GND: now also JP2.1, Q1.S, R12.1; no longer ISENS-2.KL
- net N$4: now also Q1.D, R10.1; no longer U1.VOUT
Other:
- moved on the sheet: IC3B, VIN-1, VIN-2
