File: LD Connectors/CXY1/LDConnector v3.brd (EAGLE design)
At the start: 16 x 38.1 mm, 8 parts

Commit message: updates
Parts:
- added C3, C4: 10n, rcl:C0603
- moved C2 0.16 mm to (11.0, 16.5)
Connections:
- net GND: now also C3.2, C4.2
- net N$1: now also C3.1
- net N$6: now also C4.1
Routing:
- net N$6: track 16.7 -> 17.7 mm
Changed lines of the file:
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@@
 2 NC
 3 LDA</text>
-<text x="12.065" y="15.39875" size="1.016" layer="51" font="vector" ratio="20" rot="R180">*G</text>
+<text x="9.2075" y="16.8275" size="1.016" layer="51" font="vector" ratio="20" rot="R180">*G</text>
 <text x="8.5725" y="17.145" size="1.016" layer="52" font="vector" ratio="20" rot="MR180">*A</text>
 </plain>
@@
 <element name="U$1" library="laser diode" package="TYPEA" value="LD-A" x="12.3825" y="19.05" rot="R180"/>
 <element name="U$2" library="laser diode" package="TYPEG" value="LD-G" x="16.03375" y="19.05"/>
-<element name="C2" library="rcl" package="C0603" value="0.1uF" x="10.95375" y="16.35125" rot="R180"/>
+<element name="C2" library="rcl" package="C0603" value="0.1uF" x="10.95375" y="16.51" rot="R180"/>
+<element name="C3" library="rcl" package="C0603" value="10n" x="9.525" y="16.35125" rot="MR0"/>
+<element name="C4" library="rcl" package="C0603" value="10n" x="10.95375" y="14.76375" rot="R180"/>
 </elements>
 <signals>
@@
 <via x="5.08" y="6.35" extent="1-16" drill="0.6"/>
 <contactref element="C2" pad="2"/>
+<contactref element="C3" pad="2"/>
+<contactref element="C4" pad="2"/>
 <wire x1="2.1154" y1="23.8146" x2="2.1154" y2="23.8146" width="0" layer="19" extent="1-16"/>
 </signal>
@@
 <contactref element="U$1" pad="2-PDC-LDA"/>
 <wire x1="11.43" y1="19.05" x2="14.1825" y2="19.05" width="0.8128" layer="16"/>
+<contactref element="C3" pad="1"/>
+<wire x1="10.375" y1="17.995" x2="10.375" y2="16.35125" width="0" layer="19" extent="16-16"/>
 </signal>
 <signal name="N$2">
@@
 <contactref element="U$2" pad="3-LDA"/>
 <contactref element="C2" pad="1"/>
-<wire x1="11.80375" y1="16.35125" x2="11.80375" y2="15.29625" width="0.8128" layer="1"/>
-<wire x1="11.80375" y1="15.29625" x2="4.60375" y2="8.09625" width="0.8128" layer="1"/>
+<wire x1="11.80375" y1="16.51" x2="11.80375" y2="14.76375" width="0.8128" layer="1"/>
 <wire x1="4.60375" y1="8.09625" x2="2.69875" y2="8.09625" width="0.8128" layer="1"/>
 <wire x1="14.1825" y1="17.78" x2="12.22375" y2="17.78" width="0.8128" layer="1"/>
-<wire x1="11.80375" y1="16.35125" x2="11.80375" y2="17.36" width="0.8128" layer="1"/>
+<wire x1="11.80375" y1="16.51" x2="11.80375" y2="17.36" width="0.8128" layer="1"/>
 <wire x1="11.80375" y1="17.36" x2="12.22375" y2="17.78" width="0.8128" layer="1"/>
+<contactref element="C4" pad="1"/>
+<wire x1="11.80375" y1="14.76375" x2="11.80375" y2="13.55" width="0.8128" layer="1"/>
+<wire x1="11.80375" y1="13.55" x2="10.95375" y2="12.7" width="0.8128" layer="1"/>
+<wire x1="10.95375" y1="12.7" x2="9.2075" y2="12.7" width="0.8128" layer="1"/>
+<wire x1="9.2075" y1="12.7" x2="4.60375" y2="8.09625" width="0.8128" layer="1"/>
 <wire x1="14.1825" y1="17.78" x2="14.23375" y2="17.78" width="0" layer="19" extent="1-1"/>
 </signal>
